File: Hardware-Layout-Files/MORPH RECONPLAT.sch (EAGLE design)
At the start: 16 parts, among them M1 ELECTRET_MICROPHON-WM-64PC/64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, T1 BC547, T2 BPX81

Commit message: Layout Upldate
Other:
- note removed: "Power and debugging"
- moved on the sheet: C1, C2, R6, R7, R8, T1
Changed lines of the file:
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@@
 <?xml version="1.0" encoding="utf-8"?>
 <!DOCTYPE eagle SYSTEM "eagle.dtd">
-<eagle version="6.5.0">
+<eagle version="7.1.0">
 <drawing>
 <settings>
@@
 </layers>
 <schematic xreflabel="%F%N/%S.%C%R" xrefpart="/%S.%C%R">
+<description>The Layout of Reconfigurable Platform. Developed by Daniel Graham
+LENS LAB The College of William and Mary</description>
 <attributes>
+<attribute name="DESCRIPTION" value="The Layout of Reconfigurable Platform. Developed by Daniel Graham
+LENS LAB The College of William and Mary
+"/>
+<attribute name="DRAWING_AUTHOR" value="Daniel Graham LENS LAB W&amp;N"/>
+<attribute name="TITLE" value="Reconfigurable Platform"/>
 </attributes>
 <variantdefs>
@@
 <part name="PWD" library="con-lstb" deviceset="MA03-1" device=""/>
 <part name="T2" library="opto-trans-siemens" deviceset="BPX81" device=""/>
+<part name="FRAME1" library="frames" deviceset="A4L-LOC" device="" value="DANIEL GRAHAM"/>
 </parts>
 <sheets>
 <sheet>
+<description>The Layout of Reconfigurable Platform. Developed by Daniel Graham
+LENS LAB The College of William and Mary</description>
 <plain>
-<text x="0" y="132.08" size="2.54" layer="91">Microphone and Amplifier circuit</text>
+<text x="17.78" y="127" size="2.54" layer="91">Microphone and Amplifier circuit</text>
 <text x="116.84" y="10.16" size="2.54" layer="91">Exernal Connector For Programming</text>
-<text x="129.54" y="-17.78" size="1.778" layer="91">Power and debugging</text>
 </plain>
 <instances>
@@
 <instance part="S2" gate="1" x="165.1" y="71.12"/>
 <instance part="LCD" gate="1" x="27.94" y="-22.86"/>
-<instance part="M1" gate="G$1" x="104.14" y="111.76"/>
-<instance part="R6" gate="G$1" x="99.06" y="121.92" rot="R90"/>
-<instance part="C1" gate="G$1" x="83.82" y="111.76" rot="R270"/>
-<instance part="R7" gate="G$1" x="33.02" y="111.76"/>
-<instance part="R8" gate="G$1" x="55.88" y="111.76"/>
-<instance part="C2" gate="G$1" x="35.56" y="96.52" rot="R270"/>
-<instance part="T1" gate="G$1" x="68.58" y="99.06" rot="MR270"/>
+<instance part="M1" gate="G$1" x="86.36" y="111.76" rot="MR0"/>
+<instance part="R6" gate="G$1" x="91.44" y="119.38" rot="MR90"/>
+<instance part="C1" gate="G$1" x="106.68" y="111.76" rot="MR270"/>
+<instance part="R7" gate="G$1" x="134.62" y="116.84" rot="MR270"/>
+<instance part="R8" gate="G$1" x="124.46" y="111.76" rot="MR0"/>
+<instance part="C2" gate="G$1" x="144.78" y="111.76" rot="MR270"/>
+<instance part="T1" gate="G$1" x="121.92" y="101.6"/>
 <instance part="BT" gate="1" x="-2.54" y="22.86"/>
 <instance part="DP" gate="1" x="127" y="30.48"/>
 <instance part="PWD" gate="G$1" x="114.3" y="-7.62"/>
 <instance part="T2" gate="1" x="-33.02" y="55.88"/>
+<instance part="FRAME1" gate="G$1" x="-40.64" y="-38.1"/>
 </instances>
 <busses>
@@
 </segment>
 <segment>
-<pinref part="M1" gate="G$1" pin="2"/>
-<wire x1="99.06" y1="109.22" x2="99.06" y2="101.6" width="0.1524" layer="91"/>
-<label x="99.06" y="101.6" size="1.778" layer="95" rot="R270" xref="yes"/>
-</segment>
-<segment>
-<wire x1="73.66" y1="96.52" x2="76.2" y2="96.52" width="0.1524" layer="91"/>
-<label x="76.2" y="96.52" size="1.27" layer="95" xref="yes"/>
+<wire x1="124.46" y1="96.52" x2="124.46" y2="93.98" width="0.1524" layer="91"/>
+<label x="124.46" y="93.98" size="1.27" layer="95" rot="R270" xref="yes"/>
 <pinref part="T1" gate="G$1" pin="E"/>
 </segment>
@@
 <label x="10.16" y="17.78" size="1.016" layer="95" xref="yes"/>
 <pinref part="BT" gate="1" pin="1"/>
+</segment>
+<segment>
+<pinref part="M1" gate="G$1" pin="2"/>
+<wire x1="91.44" y1="109.22" x2="91.44" y2="96.52" width="0.1524" layer="91"/>
+<label x="91.44" y="96.52" size="1.27" layer="95" rot="R270" xref="yes"/>
 </segment>
 </net>
@@
 <segment>
 <pinref part="R6" gate="G$1" pin="2"/>
-<wire x1="99.06" y1="127" x2="99.06" y2="129.54" width="0.1524" layer="91"/>
-<label x="99.06" y="129.54" size="1.27" layer="95" rot="R90" xref="yes"/>
+<wire x1="91.44" y1="124.46" x2="91.44" y2="127" width="0.1524" layer="91"/>
+<label x="91.44" y="127" size="1.27" layer="95" rot="R90" xref="yes"/>
 </segment>
 <segment>
 <pinref part="R7" gate="G$1" pin="1"/>
-<wire x1="27.94" y1="111.76" x2="20.32" y2="111.76" width="0.1524" layer="91"/>
-<label x="20.32" y="111.76" size="1.27" layer="95" rot="R180" xref="yes"/>
+<wire x1="134.62" y1="121.92" x2="134.62" y2="127" width="0.1524" layer="91"/>
+<label x="134.62" y="127" size="1.27" layer="95" rot="MR90" xref="yes"/>
 </segment>
 <segment>
@@
 </segment>
 <segment>
-<label x="22.86" y="96.52" size="1.27" layer="95" rot="R180" xref="yes"/>
+<label x="157.48" y="111.76" size="1.27" layer="95" rot="MR180" xref="yes"/>
 <pinref part="C2" gate="G$1" pin="2"/>
-<wire x1="30.48" y1="96.52" x2="22.86" y2="96.52" width="0.1524" layer="91"/>
+<wire x1="149.86" y1="111.76" x2="157.48" y2="111.76" width="0.1524" layer="91"/>
 </segment>
 </net>
@@
 <pinref part="S2" gate="1" pin="S"/>
 <wire x1="165.1" y1="76.2" x2="165.1" y2="83.82" width="0.1524" layer="91"/>
-<wire x1="165.1" y1="83.82" x2="144.78" y2="83.82" width="0.1524" layer="91"/>
-<label x="144.78" y="83.82" size="1.27" layer="95" rot="R180" xref="yes"/>
+<wire x1="165.1" y1="83.82" x2="162.56" y2="83.82" width="0.1524" layer="91"/>
+<label x="162.56" y="83.82" size="1.27" layer="95" rot="R180" xref="yes"/>
 </segment>
 </net>
@@
 <pinref part="M1" gate="G$1" pin="1"/>
 <pinref part="R6" gate="G$1" pin="1"/>
-<wire x1="99.06" y1="116.84" x2="99.06" y2="111.76" width="0.1524" layer="91"/>
+<wire x1="91.44" y1="114.3" x2="91.44" y2="111.76" width="0.1524" layer="91"/>
 <pinref part="C1" gate="G$1" pin="1"/>
-<wire x1="99.06" y1="111.76" x2="86.36" y2="111.76" width="0.1524" layer="91"/>
-<junction x="99.06" y="111.76"/>
+<wire x1="91.44" y1="111.76" x2="104.14" y2="111.76" width="0.1524" layer="91"/>
+<junction x="91.44" y="111.76"/>
 </segment>
 </net>
@@
 <segment>
 <pinref part="C1" gate="G$1" pin="2"/>
-<wire x1="78.74" y1="111.76" x2="68.58" y2="111.76" width="0.1524" layer="91"/>
+<wire x1="111.76" y1="111.76" x2="119.38" y2="111.76" width="0.1524" layer="91"/>
 <pinref part="R8" gate="G$1" pin="2"/>
 <pinref part="T1" gate="G$1" pin="B"/>
-<wire x1="68.58" y1="111.76" x2="60.96" y2="111.76" width="0.1524" layer="91"/>
-<wire x1="68.58" y1="101.6" x2="68.58" y2="111.76" width="0.1524" layer="91"/>
+<wire x1="119.38" y1="101.6" x2="119.38" y2="111.76" width="0.1524" layer="91"/>
 </segment>
 </net>
@@
 <segment>
 <pinref part="C2" gate="G$1" pin="1"/>
-<pinref part="T1" gate="G$1" pin="C"/>
-<wire x1="43.18" y1="96.52" x2="38.1" y2="96.52" width="0.1524" layer="91"/>
+<wire x1="134.62" y1="111.76" x2="142.24" y2="111.76" width="0.1524" layer="91"/>
 <pinref part="R7" gate="G$1" pin="2"/>
 <pinref part="R8" gate="G$1" pin="1"/>
-<wire x1="43.18" y1="96.52" x2="63.5" y2="96.52" width="0.1524" layer="91"/>
-<wire x1="38.1" y1="111.76" x2="43.18" y2="111.76" width="0.1524" layer="91"/>
-<wire x1="43.18" y1="111.76" x2="50.8" y2="111.76" width="0.1524" layer="91"/>
-<wire x1="43.18" y1="96.52" x2="43.18" y2="111.76" width="0.1524" layer="91"/>
-</segment>
-</net>
+<wire x1="134.62" y1="111.76" x2="129.54" y2="111.76" width="0.1524" layer="91"/>
+<junction x="134.62" y="111.76"/>
+<pinref part="T1" gate="G$1" pin="C"/>
+<wire x1="124.46" y1="106.68" x2="134.62" y2="106.68" width="0.1524" layer="91"/>
+<wire x1="134.62" y1="106.68" x2="134.62" y2="111.76" width="0.1524" layer="91"/>
+</segment>
+</net>
